File: docs/hardware/kicad/WeatherStation/WeatherStation.kicad_sch (KiCad schematic)
At the start: 12 parts, among them U1 ESP32 DevKit V1, U2 BMP280 0x76, U3 SHT45 0x44, U4 VEML7700 0x10, U5 INMP441

Commit message: docs(hardware): station takes 5 V on VIN through the base board
Other:
- note added: "5 V USB charger → DC connector on the box → base board J2 → DevKit VIN"
- note removed: "5 V USB charger feeds the DevKit Micro USB port"
Changed lines of the file:
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@@
 		(rev "3")
 	)
-	(text "5 V USB charger feeds the DevKit Micro USB port"
+	(text "5 V USB charger → DC connector on the box\n→ base board J2 → DevKit VIN"
 		(exclude_from_sim no)
 		(at 17.78 76.2 0)
