File: docs/hardware/kicad/BaseBoard/BaseBoard.kicad_sch (KiCad schematic)
At the start: 10 parts, among them J1 FTP cable, J2 5V in, U1 ESP32 DevKit V1, U2 BMP280 0x76

Commit message: feat(kicad): SPS30 UART header on the base board, runs as solder bridges
Parts:
- added J3: SPS30 cable, BaseBoard:PinHeader_1x07, symbol BaseBoard:SPS30_7_Pins
Connections:
- net +5V: now also J3.7 (5V)
- net GND: now also J3.1 (DRAIN), J3.2 (GND), J3.4 (GND), J3.6 (GND)
- new net SPS_RX: J3.3 (RX), U1.30 (D23/TX)
- new net SPS_TX: J3.5 (TX), U1.21 (D16/RX)
Other:
- note added: "J3: 4 m FTP cable to the SPS30 in the second shield. Pin order on the board: drain GND RX GND TX GND 5V."
- note added: "Runs on the board are solder bridges plus one 0R link; they are wiring, not parts, and stay off this sheet."
- note added: "SPS30 UART2 at 115200: GPIO23 to sensor RX, sensor TX to GPIO16; SEL left open (UART). Drain grounded here only."
- note removed: "Runs on the board are 0R links and solder bridges; they are wiring, not parts, and stay off this sheet."
Changed lines of the file:
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@@
 (kicad_sch (version 20250114) (generator "eeschema") (generator_version "9.0")
  (paper "A4")
-  (title_block (title "ESP32 base board on 60 x 80 mm perfboard") (date "2026-09-30") (rev "1"))
+  (title_block (title "ESP32 base board on 60 x 80 mm perfboard") (date "2026-10-15") (rev "2"))
 (symbol (lib_id "BaseBoard:DevKit_V1_BaseBoard") (at 63.5 101.6 0) (unit 1) (exclude_from_sim no) (in_bom yes) (on_board yes) (dnp no)
   (property "Reference" "U1" (at 63.5 81.28 0) (effects (font (size 1.27 1.27))))
@@
   (pin "8")
   (pin "9")
+  (pin "30")
+  (pin "21")
   (instances (project "BaseBoard" (path "/3f0c6d52-8a41-5c1e-9d37-5b2f0e4a7c19" (reference "U1") (unit 1))))
 )
@@
   (instances (project "BaseBoard" (path "/3f0c6d52-8a41-5c1e-9d37-5b2f0e4a7c19" (reference "#PWR12") (unit 1))))
 )
+(wire (pts (xy 48.26 106.68) (xy 38.1 106.68)) (stroke (width 0) (type default)))
+(label "SPS_RX" (at 38.1 106.68 0) (effects (font (size 1.27 1.27)) (justify left bottom)))
+(wire (pts (xy 48.26 109.22) (xy 38.1 109.22)) (stroke (width 0) (type default)))
+(label "SPS_TX" (at 38.1 109.22 0) (effects (font (size 1.27 1.27)) (justify left bottom)))
+(symbol (lib_id "BaseBoard:SPS30_7_Pins") (at 200.66 132.08 0) (unit 1) (exclude_from_sim no) (in_bom yes) (on_board yes) (dnp no)
+  (property "Reference" "J3" (at 198.12 120.65 0) (effects (font (size 1.27 1.27)) (justify left)))
+  (property "Value" "SPS30 cable" (at 198.12 143.51 0) (effects (font (size 1.27 1.27)) (justify left)))
+  (property "Footprint" "BaseBoard:PinHeader_1x07" (at 200.66 132.08 0) (effects (font (size 1.27 1.27)) (hide yes)))
+  (property "Datasheet" "" (at 200.66 132.08 0) (effects (font (size 1.27 1.27)) (hide yes)))
+  (pin "7")
+  (pin "3")
+  (pin "5")
+  (pin "2")
+  (pin "4")
+  (pin "6")
+  (pin "1")
+  (instances (project "BaseBoard" (path "/3f0c6d52-8a41-5c1e-9d37-5b2f0e4a7c19" (reference "J3") (unit 1))))
+)
+(wire (pts (xy 195.58 124.46) (xy 193.04 124.46)) (stroke (width 0) (type default)))
+(symbol (lib_id "BaseBoard:+5V") (at 193.04 124.46 0) (unit 1) (exclude_from_sim no) (in_bom no) (on_board no) (dnp no)
+  (property "Reference" "#PWR13" (at 193.04 128.27 0) (effects (font (size 1.27 1.27)) (hide yes)))
+  (property "Value" "+5V" (at 193.04 120.904 0) (effects (font (size 1.27 1.27))))
+  (property "Footprint" "" (at 193.04 124.46 0) (effects (font (size 1.27 1.27)) (hide yes)))
+  (property "Datasheet" "" (at 193.04 124.46 0) (effects (font (size 1.27 1.27)) (hide yes)))
+  (pin "1")
+  (instances (project "BaseBoard" (path "/3f0c6d52-8a41-5c1e-9d37-5b2f0e4a7c19" (reference "#PWR13") (unit 1))))
+)
+(wire (pts (xy 195.58 127) (xy 182.88 127)) (stroke (width 0) (type default)))
+(label "SPS_RX" (at 182.88 127 0) (effects (font (size 1.27 1.27)) (justify left bottom)))
+(wire (pts (xy 195.58 129.54) (xy 182.88 129.54)) (stroke (width 0) (type default)))
+(label "SPS_TX" (at 182.88 129.54 0) (effects (font (size 1.27 1.27)) (justify left bottom)))
+(wire (pts (xy 195.58 132.08) (xy 193.04 132.08)) (stroke (width 0) (type default)))
+(wire (pts (xy 193.04 132.08) (xy 193.04 139.7)) (stroke (width 0) (type default)))
+(wire (pts (xy 193.04 139.7) (xy 195.58 139.7)) (stroke (width 0) (type default)))
+(wire (pts (xy 195.58 134.62) (xy 193.04 134.62)) (stroke (width 0) (type default)))
+(junction (at 193.04 134.62) (diameter 0) (color 0 0 0 0))
+(wire (pts (xy 195.58 137.16) (xy 193.04 137.16)) (stroke (width 0) (type default)))
+(junction (at 193.04 137.16) (diameter 0) (color 0 0 0 0))
+(junction (at 193.04 139.7) (diameter 0) (color 0 0 0 0))
+(symbol (lib_id "BaseBoard:GND") (at 193.04 139.7 0) (unit 1) (exclude_from_sim no) (in_bom no) (on_board no) (dnp no)
+  (property "Reference" "#PWR14" (at 193.04 146.05 0) (effects (font (size 1.27 1.27)) (hide yes)))
+  (property "Value" "GND" (at 193.04 143.51 0) (effects (font (size 1.27 1.27))))
+  (property "Footprint" "" (at 193.04 139.7 0) (effects (font (size 1.27 1.27)) (hide yes)))
+  (property "Datasheet" "" (at 193.04 139.7 0) (effects (font (size 1.27 1.27)) (hide yes)))
+  (pin "1")
+  (instances (project "BaseBoard" (path "/3f0c6d52-8a41-5c1e-9d37-5b2f0e4a7c19" (reference "#PWR14") (unit 1))))
+)
 (symbol (lib_id "BaseBoard:C") (at 78.74 132.08 0) (unit 1) (exclude_from_sim no) (in_bom yes) (on_board yes) (dnp no)
   (property "Reference" "C1" (at 82.55 130.81 0) (effects (font (size 1.27 1.27)) (justify left)))
@@
 )
 (symbol (lib_id "BaseBoard:+3V3") (at 78.74 128.27 0) (unit 1) (exclude_from_sim no) (in_bom no) (on_board no) (dnp no)
-  (property "Reference" "#PWR13" (at 78.74 132.08 0) (effects (font (size 1.27 1.27)) (hide yes)))
+  (property "Reference" "#PWR15" (at 78.74 132.08 0) (effects (font (size 1.27 1.27)) (hide yes)))
   (property "Value" "+3V3" (at 78.74 124.714 0) (effects (font (size 1.27 1.27))))
   (property "Footprint" "" (at 78.74 128.27 0) (effects (font (size 1.27 1.27)) (hide yes)))
   (property "Datasheet" "" (at 78.74 128.27 0) (effects (font (size 1.27 1.27)) (hide yes)))
   (pin "1")
-  (instances (project "BaseBoard" (path "/3f0c6d52-8a41-5c1e-9d37-5b2f0e4a7c19" (reference "#PWR13") (unit 1))))
+  (instances (project "BaseBoard" (path "/3f0c6d52-8a41-5c1e-9d37-5b2f0e4a7c19" (reference "#PWR15") (unit 1))))
 )
 (symbol (lib_id "BaseBoard:GND") (at 78.74 135.89 0) (unit 1) (exclude_from_sim no) (in_bom no) (on_board no) (dnp no)
-  (property "Reference" "#PWR14" (at 78.74 142.24 0) (effects (font (size 1.27 1.27)) (hide yes)))
+  (property "Reference" "#PWR16" (at 78.74 142.24 0) (effects (font (size 1.27 1.27)) (hide yes)))
   (property "Value" "GND" (at 78.74 139.7 0) (effects (font (size 1.27 1.27))))
   (property "Footprint" "" (at 78.74 135.89 0) (effects (font (size 1.27 1.27)) (hide yes)))
   (property "Datasheet" "" (at 78.74 135.89 0) (effects (font (size 1.27 1.27)) (hide yes)))
   (pin "1")
-  (instances (project "BaseBoard" (path "/3f0c6d52-8a41-5c1e-9d37-5b2f0e4a7c19" (reference "#PWR14") (unit 1))))
+  (instances (project "BaseBoard" (path "/3f0c6d52-8a41-5c1e-9d37-5b2f0e4a7c19" (reference "#PWR16") (unit 1))))
 )
 (symbol (lib_id "BaseBoard:C_Polarized") (at 93.98 132.08 0) (unit 1) (exclude_from_sim no) (in_bom yes) (on_board yes) (dnp no)
@@
 )
 (symbol (lib_id "BaseBoard:+3V3") (at 93.98 128.27 0) (unit 1) (exclude_from_sim no) (in_bom no) (on_board no) (dnp no)
-  (property "Reference" "#PWR15" (at 93.98 132.08 0) (effects (font (size 1.27 1.27)) (hide yes)))
+  (property "Reference" "#PWR17" (at 93.98 132.08 0) (effects (font (size 1.27 1.27)) (hide yes)))
   (property "Value" "+3V3" (at 93.98 124.714 0) (effects (font (size 1.27 1.27))))
   (property "Footprint" "" (at 93.98 128.27 0) (effects (font (size 1.27 1.27)) (hide yes)))
   (property "Datasheet" "" (at 93.98 128.27 0) (effects (font (size 1.27 1.27)) (hide yes)))
   (pin "1")
-  (instances (project "BaseBoard" (path "/3f0c6d52-8a41-5c1e-9d37-5b2f0e4a7c19" (reference "#PWR15") (unit 1))))
+  (instances (project "BaseBoard" (path "/3f0c6d52-8a41-5c1e-9d37-5b2f0e4a7c19" (reference "#PWR17") (unit 1))))
 )
 (symbol (lib_id "BaseBoard:GND") (at 93.98 135.89 0) (unit 1) (exclude_from_sim no) (in_bom no) (on_board no) (dnp no)
-  (property "Reference" "#PWR16" (at 93.98 142.24 0) (effects (font (size 1.27 1.27)) (hide yes)))
+  (property "Reference" "#PWR18" (at 93.98 142.24 0) (effects (font (size 1.27 1.27)) (hide yes)))
   (property "Value" "GND" (at 93.98 139.7 0) (effects (font (size 1.27 1.27))))
   (property "Footprint" "" (at 93.98 135.89 0) (effects (font (size 1.27 1.27)) (hide yes)))
   (property "Datasheet" "" (at 93.98 135.89 0) (effects (font (size 1.27 1.27)) (hide yes)))
   (pin "1")
-  (instances (project "BaseBoard" (path "/3f0c6d52-8a41-5c1e-9d37-5b2f0e4a7c19" (reference "#PWR16") (unit 1))))
+  (instances (project "BaseBoard" (path "/3f0c6d52-8a41-5c1e-9d37-5b2f0e4a7c19" (reference "#PWR18") (unit 1))))
 )
 (label "SCL" (at 88.9 58.42 0) (effects (font (size 1.27 1.27)) (justify left bottom)))
@@
 (text "U1 sits in two 1x15 female headers. Its GND pins 2 and 17 meet on the DevKit." (exclude_from_sim no) (at 25.4 157.48 0) (effects (font (size 1.27 1.27)) (justify left)))
 (text "U2 plugs into a 1x6 female header. R1 and R2 plug into one 1x4 female header." (exclude_from_sim no) (at 25.4 162.56 0) (effects (font (size 1.27 1.27)) (justify left)))
-(text "Runs on the board are 0R links and solder bridges; they are wiring, not parts, and stay off this sheet." (exclude_from_sim no) (at 25.4 167.64 0) (effects (font (size 1.27 1.27)) (justify left)))
+(text "Runs on the board are solder bridges plus one 0R link; they are wiring, not parts, and stay off this sheet." (exclude_from_sim no) (at 25.4 167.64 0) (effects (font (size 1.27 1.27)) (justify left)))
 (text "J1: 4 m FTP cable to the shield hub. Pin order on the board: GND SCK WS SD 3V3 GND drain SDA SCL." (exclude_from_sim no) (at 25.4 172.72 0) (effects (font (size 1.27 1.27)) (justify left)))
 (text "Drain grounded here only; the shield hub end is cut back." (exclude_from_sim no) (at 25.4 177.8 0) (effects (font (size 1.27 1.27)) (justify left)))
+(text "J3: 4 m FTP cable to the SPS30 in the second shield. Pin order on the board: drain GND RX GND TX GND 5V." (exclude_from_sim no) (at 25.4 182.88 0) (effects (font (size 1.27 1.27)) (justify left)))
+(text "SPS30 UART2 at 115200: GPIO23 to sensor RX, sensor TX to GPIO16; SEL left open (UART). Drain grounded here only." (exclude_from_sim no) (at 25.4 187.96 0) (effects (font (size 1.27 1.27)) (justify left)))
   (sheet_instances (path "/" (page "1")))
 )
